Commit message: Migrate Husky UR3 simulator from ROS Noetic to ROS2 Humble
Major changes:
- Build system: Converted all 4 packages from catkin to ament_cmake
- Package.xml: Updated to format 3 with ROS2 dependencies
- C++ code: Migrated gazebo_rh_pub.cpp from roscpp to rclcpp
- Python scripts: Migrated control scripts from rospy to rclpy
- URDF/Xacro: Added ros2_control hardware interfaces
- Gazebo plugins: Updated to ROS2 compatible plugins
  - libgazebo_ros_control.so -> libgazebo_ros2_control.so
  - libgazebo_ros_laser.so -> libgazebo_ros_ray_sensor.so
  - libhector_gazebo_ros_imu.so -> libgazebo_ros_imu_sensor.so
- Navigation: Migrated from move_base to Nav2
  - gmapping replaced with slam_toolbox
  - Added nav2_params.yaml and slam_toolbox_params.yaml
- MoveIt: Updated config for MoveIt2 compatibility
- Launch files: Created new Python launch files for ROS2
  - husky_ur3_gazebo.launch.py (main simulation)
  - display.launch.py (RViz visualization)
  - navigation.launch.py (Nav2 navigation)
  - slam.launch.py (SLAM with slam_toolbox)
  - demo.launch.py (MoveIt2 demo)
- Controllers: Added ros2_controllers.yaml for ros2_control

New files:
- husky_ur3_gazebo/urdf/ros2_control.xacro
- husky_ur3_gazebo/config/ros2_controllers.yaml
- husky_ur3_navigation/config/nav2_params.yaml
- husky_ur3_navigation/config/slam_toolbox_params.yaml
- husky_ur3_gripper_moveit_config/config/ros2_controllers.yaml

Note: Legacy ROS1 launch files (*.launch) retained for reference
but new *.launch.py files should be used for ROS2

File: husky_ur3_gazebo/urdf/accessories/sick_tim571.urdf.xacro (robot description, xacro)
@@ -1,3 +1,4 @@
 <?xml version="1.0"?>
+<!-- ROS2 Humble compatible SICK TIM571 LiDAR -->
 <robot xmlns:xacro="http://www.ros.org/wiki/xacro">
   <xacro:macro name="sensor_sick_tim571" params="prefix parent prefix_topic:='front_laser' *origin min_angle:=-1.57619449019 max_angle:=1.57619449019">
@@ -33,38 +34,43 @@
     <link name="${prefix}_link">
     </link>
-    <xacro:sensor_sick_tim571_gazebo/>
+    <xacro:sensor_sick_tim571_gazebo prefix="${prefix}" prefix_topic="${prefix_topic}" min_angle="${min_angle}" max_angle="${max_angle}"/>
   </xacro:macro>
-  <xacro:macro name="sensor_sick_tim571_gazebo">
-	<gazebo reference="${prefix}_link">
-			<sensor type="ray" name="${prefix}_sensor">
-				<pose>0 0 0 0 0 0</pose>
-				<visualize>false</visualize>
-				<update_rate>15</update_rate>
-				<ray>
-					<scan>
-						<horizontal>
-							<samples>716</samples>
-							<resolution>1</resolution>
-							<min_angle>${min_angle}</min_angle>
-							<max_angle>${max_angle}</max_angle>
-						</horizontal>
-					</scan>
-					<range>
-						<min>0.05</min>
-						<max>25.0</max>
-						<resolution>0.00575</resolution>
-					</range>
-					<noise>
-						<type>gaussian</type>
-						<mean>0.0</mean>
-						<stddev>0.01</stddev>
-					</noise>
-				</ray>
-				<plugin name="${prefix}_controller" filename="libgazebo_ros_laser.so">
-					<topicName>/scan</topicName>
-					<frameName>/${prefix}_link</frameName>
-				</plugin>
-			</sensor>
-	</gazebo>
+  <xacro:macro name="sensor_sick_tim571_gazebo" params="prefix prefix_topic:='front_laser' min_angle:=-1.57619449019 max_angle:=1.57619449019">
+    <gazebo reference="${prefix}_link">
+      <sensor type="ray" name="${prefix}_sensor">
+        <pose>0 0 0 0 0 0</pose>
+        <visualize>false</visualize>
+        <update_rate>15</update_rate>
+        <ray>
+          <scan>
+            <horizontal>
+              <samples>716</samples>
+              <resolution>1</resolution>
+              <min_angle>${min_angle}</min_angle>
+              <max_angle>${max_angle}</max_angle>
+            </horizontal>
+          </scan>
+          <range>
+            <min>0.05</min>
+            <max>25.0</max>
+            <resolution>0.00575</resolution>
+          </range>
+          <noise>
+            <type>gaussian</type>
+            <mean>0.0</mean>
+            <stddev>0.01</stddev>
+          </noise>
+        </ray>
+        <!-- ROS2 Humble: Using gazebo_ros_ray_sensor plugin -->
+        <plugin name="${prefix}_controller" filename="libgazebo_ros_ray_sensor.so">
+          <ros>
+            <namespace>/</namespace>
+            <remapping>~/out:=/scan</remapping>
+          </ros>
+          <output_type>sensor_msgs/LaserScan</output_type>
+          <frame_name>${prefix}_link</frame_name>
+        </plugin>
+      </sensor>
+    </gazebo>
   </xacro:macro>
 </robot>

File: husky_ur3_gazebo/urdf/common.gazebo.xacro (robot description, xacro)
@@ -1,23 +1,12 @@
 <?xml version="1.0"?>
+<!-- ROS2 Humble compatible Gazebo configuration -->
 <robot xmlns:xacro="http://wiki.ros.org/xacro">
+  <!-- ROS2 Gazebo ros2_control plugin -->
   <gazebo>
-    <plugin name="ros_control" filename="libgazebo_ros_control.so">
-      <!--robotNamespace>/</robotNamespace-->
-      <!--robotSimType>gazebo_ros_control/DefaultRobotHWSim</robotSimType-->
+    <plugin filename="libgazebo_ros2_control.so" name="gazebo_ros2_control">
+      <robot_param>robot_description</robot_param>
+      <robot_param_node>robot_state_publisher</robot_param_node>
+      <parameters>$(find husky_ur3_gazebo)/config/ros2_controllers.yaml</parameters>
     </plugin>
-<!--
-    <plugin name="gazebo_ros_power_monitor_controller" filename="libgazebo_ros_power_monitor.so">
-      <alwaysOn>true</alwaysOn>
-      <updateRate>1.0</updateRate>
-      <timeout>5</timeout>
-      <powerStateTopic>power_state</powerStateTopic>
-      <powerStateRate>10.0</powerStateRate>
-      <fullChargeCapacity>87.78</fullChargeCapacity>
-      <dischargeRate>-474</dischargeRate>
-      <chargeRate>525</chargeRate>
-      <dischargeVoltage>15.52</dischargeVoltage>
-      <chargeVoltage>16.41</chargeVoltage>
-    </plugin>
--->
   </gazebo>
 </robot>

File: husky_ur3_gazebo/urdf/husky_ur3_gripper.urdf.xacro (robot description, xacro)
@@ -2,7 +2,8 @@
 <!--
 Software License Agreement (BSD)
-\file      husky.urdf.xacro
+\file      husky_ur3_gripper.urdf.xacro
 \authors   Paul Bovbel <pbovbel@clearpathrobotics.com>, Devon Ash <dash@clearpathrobotics.com>
 \copyright Copyright (c) 2015, Clearpath Robotics, Inc., All rights reserved.
+ROS2 Humble Migration - Updated Gazebo plugins and ros2_control
 Redistribution and use in source and binary forms, with or without modification, are permitted provided that
 the following conditions are met:
@@ -21,10 +22,10 @@
 ARISING IN ANY WAY OUT OF THE USE OF THIS SOFTWARE, EVEN IF ADVISED OF THE POSSIBILITY OF SUCH DAMAGE.
 -->
-<robot name="husky" xmlns:xacro="http://ros.org/wiki/xacro">
-  <xacro:arg name="laser_xyz" default="$(optenv HUSKY_LMS1XX_XYZ 0.3206 0.0 -0.000635)" />
-  <xacro:arg name="laser_rpy" default="$(optenv HUSKY_LMS1XX_RPY 0.0 0 0)" />
-  <xacro:property name="husky_front_bumper_extend" value="$(optenv HUSKY_FRONT_BUMPER_EXTEND 0)" />
-  <xacro:property name="husky_rear_bumper_extend" value="$(optenv HUSKY_REAR_BUMPER_EXTEND 0)" />
-  <xacro:arg name="robot_namespace" default="/husky" />
+<robot name="husky_ur3_gripper" xmlns:xacro="http://ros.org/wiki/xacro">
+  <xacro:arg name="laser_xyz" default="0.3206 0.0 -0.000635" />
+  <xacro:arg name="laser_rpy" default="0.0 0 0" />
+  <xacro:property name="husky_front_bumper_extend" value="0" />
+  <xacro:property name="husky_rear_bumper_extend" value="0" />
+  <xacro:arg name="robot_namespace" default="/" />
   <xacro:arg name="urdf_extras" default="empty.urdf" />
   <!-- Included URDF/XACRO Files -->
@@ -34,7 +35,7 @@
   <xacro:include filename="$(find husky_ur3_gazebo)/urdf/accessories/sick_tim571.urdf.xacro"/>
   <xacro:include filename="$(find husky_ur3_gazebo)/urdf/ur3_robot_gripper.urdf.xacro"/>
-  <xacro:include filename="$(find husky_ur3_gazebo)/urdf/accessories/d435_camera_h.urdf.xacro"/>-
-  <xacro:include filename="$(find husky_ur3_gazebo)/urdf/accessories/d435_camera_g.urdf.xacro"/>-
-  <!--xacro:include filename="$(find husky_ur3_gazebo)/urdf/ur3_robot.urdf.xacro"/-->
+  <xacro:include filename="$(find husky_ur3_gazebo)/urdf/accessories/d435_camera_h.urdf.xacro"/>
+  <xacro:include filename="$(find husky_ur3_gazebo)/urdf/accessories/d435_camera_g.urdf.xacro"/>
+  <xacro:include filename="$(find husky_ur3_gazebo)/urdf/ros2_control.xacro"/>
   <xacro:property name="M_PI" value="3.14159"/>
   <!-- Base Size -->
@@ -91,8 +92,7 @@
   </joint>
   <!-- IMU Link is the standard mounting position for the UM6 IMU.-->
-  <!-- Can be modified with environment variables in /etc/ros/setup.bash -->
   <link name="imu_link"/>
   <joint name="imu_joint" type="fixed">
-    <origin xyz="$(optenv HUSKY_IMU_XYZ 0.19 0 0.149)" rpy="$(optenv HUSKY_IMU_RPY 0 -1.5708 3.1416)" />
+    <origin xyz="0.19 0 0.149" rpy="0 -1.5708 3.1416" />
     <parent link="base_link" />
     <child link="imu_link" />
@@ -114,5 +114,5 @@
   </xacro:husky_wheel>
   <gazebo reference="front_left_wheel_link">
-		  <material>Gazebo/DarkGrey</material>
+      <material>Gazebo/DarkGrey</material>
       <selfCollide>false</selfCollide>
       <mu1 value="1.0"/>
@@ -121,7 +121,7 @@
       <kd value="1" />
       <fdir1 value="1 0 0"/>
-	</gazebo>
-	<gazebo reference="rear_left_wheel_link">
-		 <material>Gazebo/DarkGrey</material>
+  </gazebo>
+  <gazebo reference="rear_left_wheel_link">
+     <material>Gazebo/DarkGrey</material>
       <selfCollide>false</selfCollide>
       <mu1 value="0.05"/>
@@ -130,7 +130,7 @@
       <kd value="1" />
       <fdir1 value="1 0 0"/>
-	</gazebo>
-    <gazebo reference="front_right_wheel_link">
-		  <material>Gazebo/DarkGrey</material>
+  </gazebo>
+  <gazebo reference="front_right_wheel_link">
+      <material>Gazebo/DarkGrey</material>
       <selfCollide>false</selfCollide>
       <mu1 value="1.0"/>
@@ -139,7 +139,7 @@
       <kd value="1" />
       <fdir1 value="1 0 0"/>
-	</gazebo>
-	<gazebo reference="rear_right_wheel_link">
-		<material>Gazebo/DarkGrey</material>
+  </gazebo>
+  <gazebo reference="rear_right_wheel_link">
+    <material>Gazebo/DarkGrey</material>
       <selfCollide>false</selfCollide>
       <mu1 value="0.05"/>
@@ -148,14 +148,14 @@
       <kd value="1" />
       <fdir1 value="1 0 0"/>
-	</gazebo>
+  </gazebo>
   <xacro:husky_decorate />
   <xacro:sensor_sick_tim571 prefix="front_laser" parent="top_plate_link" prefix_topic="front_laser">
-   	<origin xyz="$(arg laser_xyz)" rpy="$(arg laser_rpy)"/>
+    <origin xyz="$(arg laser_xyz)" rpy="$(arg laser_rpy)"/>
   </xacro:sensor_sick_tim571>
- <joint name="control_box_ur3_joint" type="fixed">
-      <origin xyz="-0.095 0 0.233" rpy="${M_PI/2} 0 0" />
-      <parent link="top_plate_link"/>
-      <child link="control_box_ur3_link" />
-    </joint>
+  <joint name="control_box_ur3_joint" type="fixed">
+    <origin xyz="-0.095 0 0.233" rpy="${M_PI/2} 0 0" />
+    <parent link="top_plate_link"/>
+    <child link="control_box_ur3_link" />
+  </joint>
   <link name="control_box_ur3_link">
     <inertial>
@@ -183,37 +183,72 @@
     <material>Gazebo/DarkGrey</material>
   </gazebo>
+  <!-- ros2_control hardware interfaces -->
+  <xacro:husky_ros2_control/>
+  <xacro:ur3_ros2_control prefix=""/>
+  <xacro:gripper_ros2_control/>
+  <!-- ROS2 Gazebo ros2_control plugin -->
   <gazebo>
-    <plugin name="gazebo_ros_control" filename="libgazebo_ros_control.so">
-      <robotNamespace>$(arg robot_namespace)</robotNamespace>
+    <plugin filename="libgazebo_ros2_control.so" name="gazebo_ros2_control">
+      <robot_param>robot_description</robot_param>
+      <robot_param_node>robot_state_publisher</robot_param_node>
+      <parameters>$(find husky_ur3_gazebo)/config/ros2_controllers.yaml</parameters>
     </plugin>
   </gazebo>
-  <gazebo>
-    <plugin name="imu_controller" filename="libhector_gazebo_ros_imu.so">
-      <robotNamespace>$(arg robot_namespace)</robotNamespace>
-      <updateRate>50.0</updateRate>
-      <bodyName>base_link</bodyName>
-      <topicName>imu/data</topicName>
-      <accelDrift>0.005 0.005 0.005</accelDrift>
-      <accelGaussianNoise>0.005 0.005 0.005</accelGaussianNoise>
-      <rateDrift>0.005 0.005 0.005 </rateDrift>
-      <rateGaussianNoise>0.005 0.005 0.005 </rateGaussianNoise>
-      <headingDrift>0.005</headingDrift>
-      <headingGaussianNoise>0.005</headingGaussianNoise>
-    </plugin>
-  </gazebo>
-  <gazebo>
-    <plugin name="gps_controller" filename="libhector_gazebo_ros_gps.so">
-      <robotNamespace>$(arg robot_namespace)</robotNamespace>
-      <updateRate>40</updateRate>
-      <bodyName>base_link</bodyName>
-      <frameId>base_link</frameId>
-      <topicName>navsat/fix</topicName>
-      <velocityTopicName>navsat/vel</velocityTopicName>
-      <referenceLatitude>49.9</referenceLatitude>
-      <referenceLongitude>8.9</referenceLongitude>
-      <referenceHeading>0</referenceHeading>
-      <referenceAltitude>0</referenceAltitude>
-      <drift>0.0001 0.0001 0.0001</drift>
-    </plugin>
+  <!-- ROS2 IMU sensor plugin -->
+  <gazebo reference="imu_link">
+    <sensor name="imu_sensor" type="imu">
+      <always_on>true</always_on>
+      <update_rate>50</update_rate>
+      <imu>
+        <angular_velocity>
+          <x>
+            <noise type="gaussian">
+              <mean>0.0</mean>
+              <stddev>0.005</stddev>
+            </noise>
+          </x>
+          <y>
+            <noise type="gaussian">
+              <mean>0.0</mean>
+              <stddev>0.005</stddev>
+            </noise>
+          </y>
+          <z>
+            <noise type="gaussian">
+              <mean>0.0</mean>
+              <stddev>0.005</stddev>
+            </noise>
+          </z>
+        </angular_velocity>
+        <linear_acceleration>
+          <x>
+            <noise type="gaussian">
+              <mean>0.0</mean>
+              <stddev>0.005</stddev>
+            </noise>
+          </x>
+          <y>
+            <noise type="gaussian">
+              <mean>0.0</mean>
+              <stddev>0.005</stddev>
+            </noise>
+          </y>
+          <z>
+            <noise type="gaussian">
+              <mean>0.0</mean>
+              <stddev>0.005</stddev>
+            </noise>
+          </z>
+        </linear_acceleration>
+      </imu>
+      <plugin name="imu_plugin" filename="libgazebo_ros_imu_sensor.so">
+        <ros>
+          <namespace>/</namespace>
+          <remapping>~/out:=imu/data</remapping>
+        </ros>
+        <initial_orientation_as_reference>false</initial_orientation_as_reference>
+        <frame_name>imu_link</frame_name>
+      </plugin>
+    </sensor>
   </gazebo>
   <!-- Optional custom includes. -->
